Commit message: UPDATE: integrate stairs in urdf and display

File: description/g1/urdf/g1_29dof_stairs.urdf (robot description, URDF)
Before this commit: robot g1_29dof, 40 links, 39 joints
Links:
- added link stairs_base
- added link stairs_step_1; collision box size=0.3 1.2 0.1; visual box size=0.3 1.2 0.1
- added link stairs_step_2; collision box size=0.3 1.2 0.2; visual box size=0.3 1.2 0.2
- added link stairs_step_3; collision box size=0.3 1.2 0.30000000000000004; visual box size=0.3 1.2 0.30000000000000004
- added link stairs_step_4; collision box size=0.3 1.2 0.4; visual box size=0.3 1.2 0.4
- added link stairs_step_5; collision box size=0.3 1.2 0.5; visual box size=0.3 1.2 0.5
- added link world
Joints:
- added joint floating_base_joint: type floating, parent world, child pelvis
- added joint stairs_base_joint: type fixed, parent world, child stairs_base, origin xyz=-1.0 0.0 0.0 rpy=0 0 3.14159
- added joint stairs_step_1_joint: type fixed, parent stairs_base, child stairs_step_1
- added joint stairs_step_2_joint: type fixed, parent stairs_base, child stairs_step_2
- added joint stairs_step_3_joint: type fixed, parent stairs_base, child stairs_step_3
- added joint stairs_step_4_joint: type fixed, parent stairs_base, child stairs_step_4
- added joint stairs_step_5_joint: type fixed, parent stairs_base, child stairs_step_5

Commit message: UPDATE: modify stair params

File: description/g1/urdf/g1_29dof_stairs.urdf (robot description, URDF)
Before this commit: robot g1_29dof, 47 links, 46 joints
Joints:
- joint stairs_base_joint: origin xyz=-1.0 0.0 0.0 rpy=0 0 3.14159 -> xyz=0.75 0.0 0.0 rpy=0 0 0.0

File: description/g1/urdf/stairs.urdf (robot description, URDF)
Before this commit: robot stairs, 6 links, 6 joints
Joints:
- joint stairs_base_joint: origin xyz=-1.0 0.0 0.0 rpy=0 0 3.14159 -> xyz=0.75 0.0 0.0 rpy=0 0 0.0
