Commit message: FEAT: proprioceptive InEKF floating-base state estimation (parallel to GT)
Integrate a contact-aided Invariant EKF (legged_state_estimator) so the centroidal MPC can obtain the base pose/velocity from the pelvis IMU + joint encoders + torque-based contact instead of the MuJoCo ground-truth body frame.
It runs in parallel and publishes its odometry for evaluation; flipping floatingBase.source to "state_estimator" makes it drive control.

- new humanoid_state_estimation/ component:
  - InekfFloatingBaseEstimator wraps LeggedStateEstimator; handles the
    controller<->estimator joint-name remap (23 MPC joints -> 29 URDF joints,
    wrists zero-filled) and the IMU<->pelvis frame conversion. The InEKF tracks
    the IMU frame (8.3 cm below the pelvis); init converts pelvis->imu and
    update converts imu->pelvis with a rigid lever-arm velocity correction.
  - contact landmarks seeded at their true per-foot FK heights (correct on flat
    ground and on stairs; terrain is never assumed flat).

- sim plumbing: pelvis_imu ros2_control sensor (gyro/accel/quat) in the xacro,
  a framequat added to the MJCF, and four heel/toe contact frames (_est) in the
  URDF (the library needs exactly 4 point contacts). mujoco_ros2_control already
  exported the IMU interfaces; no change there.

- controller: claims IMU + joint-effort interfaces when the estimator is active,
  runs it each tick, bootstraps from GT once, publishes /humanoid/state_estimate/
  odom, and consumes the estimate in build_observation only when
  floatingBase.source == "state_estimator".

- stateEstimator parameter block (frames, noise, contact-estimator, LPF cutoffs);
  floatingBase.source gains the "state_estimator" option.

- vendored legged_state_estimator (package.xml, python/examples/native off).

Tuning note: the pelvis accelerometer swings +-5 m/s^2 while standing (stiff PD/contact), so accelerometer_noise is raised to 1.5 and the accel LPF cut to 30 Hz, leaning on the contact height-anchor.

Docs: docs/humanoid_state_estimation.md (math + linked code); README floating-base section updated (the GT-body dependence is now optional).

File: description/g1/urdf/g1.ros2_control_macro.xacro (robot description, xacro)
@@ -107,4 +107,21 @@
           <state_interface name="angular_velocity.z"/>
         </sensor>
+        <!-- Pelvis IMU (raw gyro + accelerometer + orientation) for the InEKF state
+             estimator. MuJoCo sensor names come from description/g1/mujoco/g1_29dof.xml. -->
+        <sensor name="pelvis_imu">
+          <param name="mujoco_quat_sensor_name">imu-pelvis-quat</param>
+          <param name="mujoco_gyro_sensor_name">imu-pelvis-angular-velocity</param>
+          <param name="mujoco_accel_sensor_name">imu-pelvis-linear-acceleration</param>
+          <state_interface name="orientation.w"/>
+          <state_interface name="orientation.x"/>
+          <state_interface name="orientation.y"/>
+          <state_interface name="orientation.z"/>
+          <state_interface name="angular_velocity.x"/>
+          <state_interface name="angular_velocity.y"/>
+          <state_interface name="angular_velocity.z"/>
+          <state_interface name="linear_acceleration.x"/>
+          <state_interface name="linear_acceleration.y"/>
+          <state_interface name="linear_acceleration.z"/>
+        </sensor>
       </xacro:if>
       <xacro:g1_joint_ros2_control

File: description/g1/urdf/g1_29dof.urdf (robot description, URDF)
Before this commit: robot g1_29dof, 40 links, 39 joints
Links:
- added link foot_l_heel_est
- added link foot_l_toe_est
- added link foot_r_heel_est
- added link foot_r_toe_est
Joints:
- added joint foot_l_heel_est_joint: type fixed, parent left_ankle_roll_link, child foot_l_heel_est, origin xyz=-0.035 0 -0.035 rpy=0 0 0
- added joint foot_l_toe_est_joint: type fixed, parent left_ankle_roll_link, child foot_l_toe_est, origin xyz=0.105 0 -0.035 rpy=0 0 0
- added joint foot_r_heel_est_joint: type fixed, parent right_ankle_roll_link, child foot_r_heel_est, origin xyz=-0.035 0 -0.035 rpy=0 0 0
- added joint foot_r_toe_est_joint: type fixed, parent right_ankle_roll_link, child foot_r_toe_est, origin xyz=0.105 0 -0.035 rpy=0 0 0
