Commit message: DESCRIPTION: one robot URDF; TF tree world -> odom -> pelvis
- g1_29dof.urdf is the only robot URDF: pelvis-rooted, no world link or floating
  joint (the MPC and the estimators add the base in code). g1.ros2_control.xacro
  includes it instead of its placeholder chain, so /robot_description is the real
  model for both the controller manager and robot_state_publisher.
  Removed g1_29dof_stairs.urdf, the generated stairs.urdf and displayUrdfFile.
- TF: world -> odom static identity; odom -> pelvis from the estimator controller
  (real-time /tf publisher, odometry frame now odom); ground truth as
  world -> gt/pelvis, or world -> pelvis when no estimator runs.
- The stairs are an environment description rooted at world (stairs.urdf.xacro,
  same params file as the MuJoCo stairs), published by a second
  robot_state_publisher on /environment/robot_description; rviz Environment
  display. environmentDescription:="" for scenes without stairs.

Co-Authored-By: Claude Opus 5.5 <noreply@anthropic.com>

File: description/g1/urdf/g1.ros2_control.xacro (robot description, xacro)
@@ -19,239 +19,8 @@
   <xacro:property name="joint_init" value="${initial_pose['g1_joints']}"/>
   <xacro:include filename="$(find legged_robot_mpc_controller)/description/g1/urdf/g1.ros2_control_macro.xacro"/>
-  <!-- Minimal kinematic chain for ros2_control (joint names must match the URDF used by the MPC).
-       The floating base is not part of ros2_control; MuJoCo owns the free joint. -->
-  <link name="pelvis"/>
-  <link name="left_hip_pitch_link"/>
-  <link name="left_hip_roll_link"/>
-  <link name="left_hip_yaw_link"/>
-  <link name="left_knee_link"/>
-  <link name="left_ankle_pitch_link"/>
-  <link name="left_ankle_roll_link"/>
-  <link name="right_hip_pitch_link"/>
-  <link name="right_hip_roll_link"/>
-  <link name="right_hip_yaw_link"/>
-  <link name="right_knee_link"/>
-  <link name="right_ankle_pitch_link"/>
-  <link name="right_ankle_roll_link"/>
-  <link name="waist_yaw_link"/>
-  <link name="waist_roll_link"/>
-  <link name="torso_link"/>
-  <link name="left_shoulder_pitch_link"/>
-  <link name="left_shoulder_roll_link"/>
-  <link name="left_shoulder_yaw_link"/>
-  <link name="left_elbow_link"/>
-  <link name="left_wrist_roll_link"/>
-  <link name="left_wrist_pitch_link"/>
-  <link name="left_wrist_yaw_link"/>
-  <link name="right_shoulder_pitch_link"/>
-  <link name="right_shoulder_roll_link"/>
-  <link name="right_shoulder_yaw_link"/>
-  <link name="right_elbow_link"/>
-  <link name="right_wrist_roll_link"/>
-  <link name="right_wrist_pitch_link"/>
-  <link name="right_wrist_yaw_link"/>
-  <joint name="left_hip_pitch_joint" type="revolute">
-    <parent link="pelvis"/>
-    <child link="left_hip_pitch_link"/>
-    <origin xyz="0 0 0" rpy="0 0 0"/>
-    <axis xyz="0 1 0"/>
-    <limit lower="-2.5307" upper="2.8798" effort="88" velocity="32"/>
-  </joint>
-  <joint name="left_hip_roll_joint" type="revolute">
-    <parent link="left_hip_pitch_link"/>
-    <child link="left_hip_roll_link"/>
-    <origin xyz="0 0 0" rpy="0 0 0"/>
-    <axis xyz="1 0 0"/>
-    <limit lower="-0.5236" upper="2.9671" effort="88" velocity="32"/>
-  </joint>
-  <joint name="left_hip_yaw_joint" type="revolute">
-    <parent link="left_hip_roll_link"/>
-    <child link="left_hip_yaw_link"/>
-    <origin xyz="0 0 0" rpy="0 0 0"/>
-    <axis xyz="0 0 1"/>
-    <limit lower="-2.7576" upper="2.7576" effort="88" velocity="32"/>
-  </joint>
-  <joint name="left_knee_joint" type="revolute">
-    <parent link="left_hip_yaw_link"/>
-    <child link="left_knee_link"/>
-    <origin xyz="0 0 0" rpy="0 0 0"/>
-    <axis xyz="0 1 0"/>
-    <limit lower="-0.087267" upper="2.8798" effort="139" velocity="20"/>
-  </joint>
-  <joint name="left_ankle_pitch_joint" type="revolute">
-    <parent link="left_knee_link"/>
-    <child link="left_ankle_pitch_link"/>
-    <origin xyz="0 0 0" rpy="0 0 0"/>
-    <axis xyz="0 1 0"/>
-    <limit lower="-0.87267" upper="0.5236" effort="50" velocity="37"/>
-  </joint>
-  <joint name="left_ankle_roll_joint" type="revolute">
-    <parent link="left_ankle_pitch_link"/>
-    <child link="left_ankle_roll_link"/>
-    <origin xyz="0 0 0" rpy="0 0 0"/>
-    <axis xyz="1 0 0"/>
-    <limit lower="-0.2618" upper="0.2618" effort="50" velocity="37"/>
-  </joint>
-  <joint name="right_hip_pitch_joint" type="revolute">
-    <parent link="pelvis"/>
-    <child link="right_hip_pitch_link"/>
-    <origin xyz="0 0 0" rpy="0 0 0"/>
-    <axis xyz="0 1 0"/>
-    <limit lower="-2.5307" upper="2.8798" effort="88" velocity="32"/>
-  </joint>
-  <joint name="right_hip_roll_joint" type="revolute">
-    <parent link="right_hip_pitch_link"/>
-    <child link="right_hip_roll_link"/>
-    <origin xyz="0 0 0" rpy="0 0 0"/>
-    <axis xyz="1 0 0"/>
-    <limit lower="-2.9671" upper="0.5236" effort="88" velocity="32"/>
-  </joint>
-  <joint name="right_hip_yaw_joint" type="revolute">
-    <parent link="right_hip_roll_link"/>
-    <child link="right_hip_yaw_link"/>
-    <origin xyz="0 0 0" rpy="0 0 0"/>
-    <axis xyz="0 0 1"/>
-    <limit lower="-2.7576" upper="2.7576" effort="88" velocity="32"/>
-  </joint>
-  <joint name="right_knee_joint" type="revolute">
-    <parent link="right_hip_yaw_link"/>
-    <child link="right_knee_link"/>
-    <origin xyz="0 0 0" rpy="0 0 0"/>
-    <axis xyz="0 1 0"/>
-    <limit lower="-0.087267" upper="2.8798" effort="139" velocity="20"/>
-  </joint>
-  <joint name="right_ankle_pitch_joint" type="revolute">
-    <parent link="right_knee_link"/>
-    <child link="right_ankle_pitch_link"/>
-    <origin xyz="0 0 0" rpy="0 0 0"/>
-    <axis xyz="0 1 0"/>
-    <limit lower="-0.87267" upper="0.5236" effort="50" velocity="37"/>
-  </joint>
-  <joint name="right_ankle_roll_joint" type="revolute">
-    <parent link="right_ankle_pitch_link"/>
-    <child link="right_ankle_roll_link"/>
-    <origin xyz="0 0 0" rpy="0 0 0"/>
-    <axis xyz="1 0 0"/>
-    <limit lower="-0.2618" upper="0.2618" effort="50" velocity="37"/>
-  </joint>
-  <joint name="waist_yaw_joint" type="revolute">
-    <parent link="pelvis"/>
-    <child link="waist_yaw_link"/>
-    <origin xyz="0 0 0" rpy="0 0 0"/>
-    <axis xyz="0 0 1"/>
-    <limit lower="-2.618" upper="2.618" effort="88" velocity="32"/>
-  </joint>
-  <joint name="waist_roll_joint" type="revolute">
-    <parent link="waist_yaw_link"/>
-    <child link="waist_roll_link"/>
-    <origin xyz="0 0 0" rpy="0 0 0"/>
-    <axis xyz="1 0 0"/>
-    <limit lower="-0.52" upper="0.52" effort="50" velocity="37"/>
-  </joint>
-  <joint name="waist_pitch_joint" type="revolute">
-    <parent link="waist_roll_link"/>
-    <child link="torso_link"/>
-    <origin xyz="0 0 0" rpy="0 0 0"/>
-    <axis xyz="0 1 0"/>
-    <limit lower="-0.52" upper="0.52" effort="50" velocity="37"/>
-  </joint>
-  <joint name="left_shoulder_pitch_joint" type="revolute">
-    <parent link="torso_link"/>
-    <child link="left_shoulder_pitch_link"/>
-    <origin xyz="0 0 0" rpy="0 0 0"/>
-    <axis xyz="0 1 0"/>
-    <limit lower="-3.0892" upper="2.6704" effort="25" velocity="37"/>
-  </joint>
-  <joint name="left_shoulder_roll_joint" type="revolute">
-    <parent link="left_shoulder_pitch_link"/>
-    <child link="left_shoulder_roll_link"/>
-    <origin xyz="0 0 0" rpy="0 0 0"/>
-    <axis xyz="1 0 0"/>
-    <limit lower="-1.5882" upper="2.2515" effort="25" velocity="37"/>
-  </joint>
-  <joint name="left_shoulder_yaw_joint" type="revolute">
-    <parent link="left_shoulder_roll_link"/>
-    <child link="left_shoulder_yaw_link"/>
-    <origin xyz="0 0 0" rpy="0 0 0"/>
-    <axis xyz="0 0 1"/>
-    <limit lower="-2.618" upper="2.618" effort="25" velocity="37"/>
-  </joint>
-  <joint name="left_elbow_joint" type="revolute">
-    <parent link="left_shoulder_yaw_link"/>
-    <child link="left_elbow_link"/>
-    <origin xyz="0 0 0" rpy="0 0 0"/>
-    <axis xyz="0 1 0"/>
-    <limit lower="-1.0472" upper="2.0944" effort="25" velocity="37"/>
-  </joint>
-  <joint name="left_wrist_roll_joint" type="revolute">
-    <parent link="left_elbow_link"/>
-    <child link="left_wrist_roll_link"/>
-    <origin xyz="0 0 0" rpy="0 0 0"/>
-    <axis xyz="1 0 0"/>
-    <limit lower="-1.972222054" upper="1.972222054" effort="25" velocity="37"/>
-  </joint>
-  <joint name="left_wrist_pitch_joint" type="revolute">
-    <parent link="left_wrist_roll_link"/>
-    <child link="left_wrist_pitch_link"/>
-    <origin xyz="0 0 0" rpy="0 0 0"/>
-    <axis xyz="0 1 0"/>
-    <limit lower="-1.614429558" upper="1.614429558" effort="5" velocity="22"/>
-  </joint>
-  <joint name="left_wrist_yaw_joint" type="revolute">
-    <parent link="left_wrist_pitch_link"/>
-    <child link="left_wrist_yaw_link"/>
-    <origin xyz="0 0 0" rpy="0 0 0"/>
-    <axis xyz="0 0 1"/>
-    <limit lower="-1.614429558" upper="1.614429558" effort="5" velocity="22"/>
-  </joint>
-  <joint name="right_shoulder_pitch_joint" type="revolute">
-    <parent link="torso_link"/>
-    <child link="right_shoulder_pitch_link"/>
-    <origin xyz="0 0 0" rpy="0 0 0"/>
-    <axis xyz="0 1 0"/>
-    <limit lower="-3.0892" upper="2.6704" effort="25" velocity="37"/>
-  </joint>
-  <joint name="right_shoulder_roll_joint" type="revolute">
-    <parent link="right_shoulder_pitch_link"/>
-    <child link="right_shoulder_roll_link"/>
-    <origin xyz="0 0 0" rpy="0 0 0"/>
-    <axis xyz="1 0 0"/>
-    <limit lower="-2.2515" upper="1.5882" effort="25" velocity="37"/>
-  </joint>
-  <joint name="right_shoulder_yaw_joint" type="revolute">
-    <parent link="right_shoulder_roll_link"/>
-    <child link="right_shoulder_yaw_link"/>
-    <origin xyz="0 0 0" rpy="0 0 0"/>
-    <axis xyz="0 0 1"/>
-    <limit lower="-2.618" upper="2.618" effort="25" velocity="37"/>
-  </joint>
-  <joint name="right_elbow_joint" type="revolute">
-    <parent link="right_shoulder_yaw_link"/>
-    <child link="right_elbow_link"/>
-    <origin xyz="0 0 0" rpy="0 0 0"/>
-    <axis xyz="0 1 0"/>
-    <limit lower="-1.0472" upper="2.0944" effort="25" velocity="37"/>
-  </joint>
-  <joint name="right_wrist_roll_joint" type="revolute">
-    <parent link="right_elbow_link"/>
-    <child link="right_wrist_roll_link"/>
-    <origin xyz="0 0 0" rpy="0 0 0"/>
-    <axis xyz="1 0 0"/>
-    <limit lower="-1.972222054" upper="1.972222054" effort="25" velocity="37"/>
-  </joint>
-  <joint name="right_wrist_pitch_joint" type="revolute">
-    <parent link="right_wrist_roll_link"/>
-    <child link="right_wrist_pitch_link"/>
-    <origin xyz="0 0 0" rpy="0 0 0"/>
-    <axis xyz="0 1 0"/>
-    <limit lower="-1.614429558" upper="1.614429558" effort="5" velocity="22"/>
-  </joint>
-  <joint name="right_wrist_yaw_joint" type="revolute">
-    <parent link="right_wrist_pitch_link"/>
-    <child link="right_wrist_yaw_link"/>
-    <origin xyz="0 0 0" rpy="0 0 0"/>
-    <axis xyz="0 0 1"/>
-    <limit lower="-1.614429558" upper="1.614429558" effort="5" velocity="22"/>
-  </joint>
+  <!-- The robot itself: the one URDF, rooted at the pelvis. The floating base is not a
+       joint here - MuJoCo owns the free joint, the MPC and the estimator add the base in
+       code, and odom -> pelvis comes from the estimator as a TF. -->
+  <xacro:include filename="$(find legged_robot_mpc_controller)/description/g1/urdf/g1_29dof.urdf"/>
   <xacro:g1_ros2_control
     use_fake_hardware="${use_fake_hardware}"

File: description/g1/urdf/stairs.urdf.xacro (robot description, xacro)
@@ -2,18 +2,12 @@
 <robot name="stairs" xmlns:xacro="http://www.ros.org/wiki/xacro">
   <!--
-    Parametric staircase for URDF (same geometry convention as
-    ../mujoco/stairs.xml.xacro, driven by the SAME params file).
-    Generate a standalone urdf:
-      sudo xacro \
-        ./stairs.urdf.xacro \
-        stairs_params_file:=../mujoco/stairs_params.yaml \
-        parent:=world \
-        -o ./stairs.urdf
-    The result is a chain of fixed joints:
+    Environment description: a parametric staircase (same geometry convention
+    as ../mujoco/stairs.xml.xacro, driven by the SAME params file). It is not
+    part of the robot. g1.launch.py runs it through xacro and publishes it with
+    its own robot_state_publisher in the "environment" namespace, so rviz shows
+    it next to the robot.
+    The result is a chain of fixed joints, rooted at <parent> (default "world"):
       <parent> -[fixed]-> stairs_base -[fixed]-> stairs_step_1 ... stairs_step_N
     The "stairs_base" link is the 0th step reference frame (world pos + yaw).
-    To fold it into g1_29dof.urdf: copy the generated <link>/<joint> blocks in,
-    and make sure the chosen <parent> link (default "world") exists in that file
-    (g1_29dof.urdf already has a commented-out "world" link you can enable).
     Each step is a SOLID box from the ground up to its tread height; the box
     origin sits at half that height.
@@ -32,4 +26,5 @@
   <xacro:property name="gray_step" value="${stairs['color_gray_step']}"/>
   <xacro:property name="gray_max"  value="${stairs['color_gray_max']}"/>
+  <link name="${parent_link}"/>
   <!-- 0th step reference frame: world center position + yaw. -->
   <link name="stairs_base"/>

Commit message: FEAT: G1 rev_1_0 model; WB-ID writes per-joint effort_pd gains
- g1_29dof.xml / g1_29dof.urdf are now Unitree's g1_29dof_rev_1_0 (mode_machine 5,
  33.34 kg), replacing the deprecated g1_29dof (35.11 kg). MJCF joint dynamics:
  per-motor armature from unitree_rl_lab, damping 0.05 / frictionloss 0.2 (0.1 on
  wrist pitch/yaw) from unitree_mujoco, implicitfast. g1_29dof_real.xml removed.
- Hip roll is the 139 N m actuator: control.torqueLimit in both controllers and
  the ros2_control command limit.
- WB-ID: control.jointEffortPd.kp/kd per joint (1200 / 20), written to the
  <joint>/kp, <joint>/kd command interfaces every tick in every bring-up phase and
  kept on deactivation. The xacro keeps the hardware defaults (1200 / 10, wrists
  100 / 1) for centroidal, the wrists and before activation. Requires
  mujoco_ros2_control b23ee84 (kp/kd command interfaces).
- Contract test checks the gain arrays; Codex.md handoff updated.

Co-Authored-By: Claude Opus 5.5 <noreply@anthropic.com>

File: description/g1/urdf/g1.ros2_control.xacro (robot description, xacro)
@@ -5,4 +5,6 @@
   <xacro:arg name="initial_pose_file" default=""/>
   <xacro:arg name="ros2_control_command_interface" default="effort_pd"/>
+  <xacro:arg name="effort_pd_kp" default="1200.0"/>
+  <xacro:arg name="effort_pd_kd" default="10.0"/>
   <xacro:arg name="mujoco_position_kp" default="10000"/>
   <xacro:arg name="mujoco_position_ki" default="50"/>
@@ -29,4 +31,6 @@
     joint_init="${joint_init}"
     command_interface="${ros2_control_command_interface}"
+    effort_pd_kp="$(arg effort_pd_kp)"
+    effort_pd_kd="$(arg effort_pd_kd)"
     mujoco_position_kp="$(arg mujoco_position_kp)"
     mujoco_position_ki="$(arg mujoco_position_ki)"

File: description/g1/urdf/g1.ros2_control_macro.xacro (robot description, xacro)
@@ -27,4 +27,8 @@
           <param name="max">${effort_limit}</param>
         </command_interface>
+        <!-- Servo gains: start at effort_pd_kp / effort_pd_kd; a controller that claims these
+             sets them per joint (WB-ID: control.jointEffortPd). -->
+        <command_interface name="kp"/>
+        <command_interface name="kd"/>
       </xacro:if>
       <xacro:if value="${command_interface == 'effort'}">
@@ -167,4 +171,17 @@
         effort_pd_kp="${effort_pd_kp}"
         effort_pd_kd="${effort_pd_kd}"
+        effort_limit="139"
+        mujoco_position_kp="${mujoco_position_kp}"
+        mujoco_position_ki="${mujoco_position_ki}"
+        mujoco_position_kd="${mujoco_position_kd}"
+        mujoco_position_i_max="${mujoco_position_i_max}"
+        mujoco_position_i_min="${mujoco_position_i_min}"/>
+      <xacro:g1_joint_ros2_control
+        joint_name="left_hip_yaw_joint"
+        use_mujoco_sim="${use_mujoco_sim}"
+        joint_init="${joint_init}"
+        command_interface="${command_interface}"
+        effort_pd_kp="${effort_pd_kp}"
+        effort_pd_kd="${effort_pd_kd}"
         effort_limit="88"
         mujoco_position_kp="${mujoco_position_kp}"
@@ -174,5 +191,44 @@
         mujoco_position_i_min="${mujoco_position_i_min}"/>
       <xacro:g1_joint_ros2_control
-        joint_name="left_hip_yaw_joint"
+        joint_name="left_knee_joint"
+        use_mujoco_sim="${use_mujoco_sim}"
+        joint_init="${joint_init}"
+        command_interface="${command_interface}"
+        effort_pd_kp="${effort_pd_kp}"
+        effort_pd_kd="${effort_pd_kd}"
+        effort_limit="139"
+        mujoco_position_kp="${mujoco_position_kp}"
+        mujoco_position_ki="${mujoco_position_ki}"
+        mujoco_position_kd="${mujoco_position_kd}"
+        mujoco_position_i_max="${mujoco_position_i_max}"
+        mujoco_position_i_min="${mujoco_position_i_min}"/>
+      <xacro:g1_joint_ros2_control
+        joint_name="left_ankle_pitch_joint"
+        use_mujoco_sim="${use_mujoco_sim}"
+        joint_init="${joint_init}"
+        command_interface="${command_interface}"
+        effort_pd_kp="${effort_pd_kp}"
+        effort_pd_kd="${effort_pd_kd}"
+        effort_limit="50"
+        mujoco_position_kp="${mujoco_position_kp}"
+        mujoco_position_ki="${mujoco_position_ki}"
+        mujoco_position_kd="${mujoco_position_kd}"
+        mujoco_position_i_max="${mujoco_position_i_max}"
+        mujoco_position_i_min="${mujoco_position_i_min}"/>
+      <xacro:g1_joint_ros2_control
+        joint_name="left_ankle_roll_joint"
+        use_mujoco_sim="${use_mujoco_sim}"
+        joint_init="${joint_init}"
+        command_interface="${command_interface}"
+        effort_pd_kp="${effort_pd_kp}"
+        effort_pd_kd="${effort_pd_kd}"
+        effort_limit="50"
+        mujoco_position_kp="${mujoco_position_kp}"
+        mujoco_position_ki="${mujoco_position_ki}"
+        mujoco_position_kd="${mujoco_position_kd}"
+        mujoco_position_i_max="${mujoco_position_i_max}"
+        mujoco_position_i_min="${mujoco_position_i_min}"/>
+      <xacro:g1_joint_ros2_control
+        joint_name="right_hip_pitch_joint"
         use_mujoco_sim="${use_mujoco_sim}"
         joint_init="${joint_init}"
@@ -187,5 +243,5 @@
         mujoco_position_i_min="${mujoco_position_i_min}"/>
       <xacro:g1_joint_ros2_control
-        joint_name="left_knee_joint"
+        joint_name="right_hip_roll_joint"
         use_mujoco_sim="${use_mujoco_sim}"
         joint_init="${joint_init}"
@@ -194,56 +250,4 @@
         effort_pd_kd="${effort_pd_kd}"
         effort_limit="139"
-        mujoco_position_kp="${mujoco_position_kp}"
-        mujoco_position_ki="${mujoco_position_ki}"
-        mujoco_position_kd="${mujoco_position_kd}"
-        mujoco_position_i_max="${mujoco_position_i_max}"
-        mujoco_position_i_min="${mujoco_position_i_min}"/>
-      <xacro:g1_joint_ros2_control
-        joint_name="left_ankle_pitch_joint"
-        use_mujoco_sim="${use_mujoco_sim}"
-        joint_init="${joint_init}"
-        command_interface="${command_interface}"
-        effort_pd_kp="${effort_pd_kp}"
-        effort_pd_kd="${effort_pd_kd}"
-        effort_limit="50"
-        mujoco_position_kp="${mujoco_position_kp}"
-        mujoco_position_ki="${mujoco_position_ki}"
-        mujoco_position_kd="${mujoco_position_kd}"
-        mujoco_position_i_max="${mujoco_position_i_max}"
-        mujoco_position_i_min="${mujoco_position_i_min}"/>
-      <xacro:g1_joint_ros2_control
-        joint_name="left_ankle_roll_joint"
-        use_mujoco_sim="${use_mujoco_sim}"
-        joint_init="${joint_init}"
-        command_interface="${command_interface}"
-        effort_pd_kp="${effort_pd_kp}"
-        effort_pd_kd="${effort_pd_kd}"
-        effort_limit="50"
-        mujoco_position_kp="${mujoco_position_kp}"
-        mujoco_position_ki="${mujoco_position_ki}"
-        mujoco_position_kd="${mujoco_position_kd}"
-        mujoco_position_i_max="${mujoco_position_i_max}"
-        mujoco_position_i_min="${mujoco_position_i_min}"/>
-      <xacro:g1_joint_ros2_control
-        joint_name="right_hip_pitch_joint"
-        use_mujoco_sim="${use_mujoco_sim}"
-        joint_init="${joint_init}"
-        command_interface="${command_interface}"
-        effort_pd_kp="${effort_pd_kp}"
-        effort_pd_kd="${effort_pd_kd}"
-        effort_limit="88"
-        mujoco_position_kp="${mujoco_position_kp}"
-        mujoco_position_ki="${mujoco_position_ki}"
-        mujoco_position_kd="${mujoco_position_kd}"
-        mujoco_position_i_max="${mujoco_position_i_max}"
-        mujoco_position_i_min="${mujoco_position_i_min}"/>
-      <xacro:g1_joint_ros2_control
-        joint_name="right_hip_roll_joint"
-        use_mujoco_sim="${use_mujoco_sim}"
-        joint_init="${joint_init}"
-        command_interface="${command_interface}"
-        effort_pd_kp="${effort_pd_kp}"
-        effort_pd_kd="${effort_pd_kd}"
-        effort_limit="88"
         mujoco_position_kp="${mujoco_position_kp}"
         mujoco_position_ki="${mujoco_position_ki}"

File: description/g1/urdf/g1_29dof.urdf (robot description, URDF)
Before this commit: robot g1_29dof, 44 links, 43 joints
Links:
- removed link waist_support_link
- link torso_link: mass 8.562 -> 6.78
- link waist_roll_link: mass 0.047 -> 0.086
- link waist_yaw_link: mass 0.244 -> 0.214
Joints:
- removed joint waist_support_joint
- joint d435_joint: origin xyz=0.0576235 0.01753 0.41987 rpy=0 0.8307767239493009 0 -> xyz=0.0576235 0.01753 0.42987 rpy=0 0.8307767239493009 0
- joint head_joint: origin xyz=0.0039635 0 -0.054 rpy=0 0 0 -> xyz=0.0039635 0 -0.044 rpy=0 0 0
- joint imu_in_torso_joint: origin xyz=-0.03959 -0.00224 0.13792 rpy=0 0 0 -> xyz=-0.03959 -0.00224 0.14792 rpy=0 0 0
- joint left_hip_roll_joint: limit lower=-0.5236 upper=2.9671 effort=88 velocity=32 -> lower=-0.5236 upper=2.9671 effort=139 velocity=20
- joint left_shoulder_pitch_joint: origin xyz=0.0039563 0.10022 0.23778 rpy=0.27931 5.4949E-05 -0.00019159 -> xyz=0.0039563 0.10022 0.24778 rpy=0.27931 5.4949E-05 -0.00019159
- joint logo_joint: origin xyz=0.0039635 0 -0.054 rpy=0 0 0 -> xyz=0.0039635 0 -0.044 rpy=0 0 0
- joint mid360_joint: origin xyz=0.0002835 0.00003 0.40618 rpy=0 0.04014257279586953 0 -> xyz=0.0002835 0.00003 0.428434 rpy=3.141592653589793 0.05112069379091391 0
- joint right_hip_roll_joint: limit lower=-2.9671 upper=0.5236 effort=88 velocity=32 -> lower=-2.9671 upper=0.5236 effort=139 velocity=20
- joint right_shoulder_pitch_joint: origin xyz=0.0039563 -0.10021 0.23778 rpy=-0.27931 5.4949E-05 0.00019159 -> xyz=0.0039563 -0.10021 0.24778 rpy=-0.27931 5.4949E-05 0.00019159
- joint waist_pitch_joint: origin xyz=0 0 0.019 rpy=0 0 0 -> xyz=0 0 0 rpy=0 0 0
- joint waist_roll_joint: origin xyz=-0.0039635 0 0.035 rpy=0 0 0 -> xyz=-0.0039635 0 0.044 rpy=0 0 0
