Commit message: XML: reorganize robot assets and shared MuJoCo scenes
- move G1 models and meshes to description/robots/g1
- group shared environments under description/mujoco
- update launch paths, scene generator and documentation links
- add layout regression tests and verify unchanged physics

File: description/mujoco/terrains/stairs.urdf.xacro (robot description, xacro)
@@ -3,5 +3,5 @@
   <!--
     Environment description: a parametric staircase (same geometry convention
-    as ../mujoco/stairs.xml.xacro, driven by the SAME params file). It is not
+    as stairs.xml.xacro, driven by the SAME params file). It is not
     part of the robot. g1.launch.py runs it through xacro and publishes it with
     its own robot_state_publisher in the "environment" namespace, so rviz shows
@@ -13,5 +13,5 @@
     origin sits at half that height.
   -->
-  <xacro:arg name="stairs_params_file" default="../mujoco/stairs_params.yaml"/>
+  <xacro:arg name="stairs_params_file" default="stairs_params.yaml"/>
   <xacro:arg name="parent" default="world"/>
   <xacro:property name="stairs_params_file" value="$(arg stairs_params_file)"/>

File: description/robots/g1/urdf/g1.ros2_control.xacro (robot description, xacro)
@@ -14,5 +14,5 @@
   <xacro:arg name="mujoco_effort_command_mode" default="actuator"/>
   <xacro:arg name="use_lidar" default="false"/>
-  <xacro:arg name="robot_urdf_file" default="$(find legged_robot_mpc_controller)/description/g1/urdf/g1_29dof.urdf"/>
+  <xacro:arg name="robot_urdf_file" default="$(find legged_robot_mpc_controller)/description/robots/g1/urdf/g1_29dof.urdf"/>
   <xacro:property name="use_fake_hardware" value="$(arg use_fake_hardware)"/>
   <xacro:property name="use_mujoco_sim" value="$(arg use_mujoco_sim)"/>
@@ -21,5 +21,5 @@
   <xacro:property name="initial_pose" value="${xacro.load_yaml(initial_pose_file)}"/>
   <xacro:property name="joint_init" value="${initial_pose['g1_joints']}"/>
-  <xacro:include filename="$(find legged_robot_mpc_controller)/description/g1/urdf/g1.ros2_control_macro.xacro"/>
+  <xacro:include filename="$(find legged_robot_mpc_controller)/description/robots/g1/urdf/g1.ros2_control_macro.xacro"/>
   <!-- The robot itself: the one URDF, rooted at the pelvis. The floating base is not a
        joint here - MuJoCo owns the free joint, the MPC and the estimator add the base in

File: description/robots/g1/urdf/g1.ros2_control_macro.xacro (robot description, xacro)
@@ -119,5 +119,5 @@
         </sensor>
         <!-- Pelvis IMU (raw gyro + accelerometer + orientation) for the InEKF state
-             estimator. MuJoCo sensor names come from description/g1/mujoco/g1_29dof.xml. -->
+             estimator. MuJoCo sensor names come from description/robots/g1/mujoco/g1_29dof.xml. -->
         <sensor name="pelvis_imu">
           <param name="mujoco_quat_sensor_name">imu-pelvis-quat</param>

File: description/robots/g1/urdf/g1_29dof.urdf (robot description, URDF)
Before this commit: robot g1_29dof, 43 links, 42 joints
Links:
- link head_link: geometry collision mesh filename=package://legged_robot_mpc_controller/description/robots/g1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; visual mesh filename=package://legged_robot_mpc_controller/description/robots/g1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
- link left_ankle_pitch_link: geometry collision mesh filename=package://legged_robot_mpc_controller/description/robots/g1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; visual mesh filename=package://legged_robot_mpc_controller/description/robots/g1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
- link left_ankle_roll_link: geometry collision sphere radius=0.005; collision sphere radius=0.005
- link left_elbow_link: geometry collision mesh filename=package://legged_robot_mpc_controller/description/robots/g1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; visual mesh filename=package://legged_robot_mpc_controller/description/robots/g1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
- link left_hip_pitch_link: geometry collision mesh filename=package://legged_robot_mpc_controller/description/robots/g1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; visual mesh filename=package://legged_robot_mpc_controller/description/robots/g1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
- link left_hip_roll_link: geometry collision mesh filename=package://legged_robot_mpc_controller/description/robots/g1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; visual mesh filename=package://legged_robot_mpc_controller/description/robots/g1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
- link left_hip_yaw_link: geometry collision mesh filename=package://legged_robot_mpc_controller/description/robots/g1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; visual mesh filename=package://legged_robot_mpc_controller/description/robots/g1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
- link left_knee_link: geometry collision mesh filename=package://legged_robot_mpc_controller/description/robots/g1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; visual mesh filename=package://legged_robot_mpc_controller/description/robots/g1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
- link left_rubber_hand: geometry visual mesh filename=package://legged_robot_mpc_controller/description/robots/g1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
- link left_shoulder_pitch_link: geometry collision cylinder length=0.05 radius=0.03; visual mesh filename=package://legged_robot_mpc_controller/description/robots/g1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
- link left_shoulder_roll_link: geometry collision cylinder length=0.03 radius=0.03; visual mesh filename=package://legged_robot_mpc_controller/description/robots/g1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
- link left_shoulder_yaw_link: geometry collision mesh filename=package://legged_robot_mpc_controller/description/robots/g1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; visual mesh filename=package://legged_robot_mpc_controller/description/robots/g1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
- link left_wrist_pitch_link: geometry collision mesh filename=package://legged_robot_mpc_controller/description/robots/g1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; visual mesh filename=package://legged_robot_mpc_controller/description/robots/g1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
- link left_wrist_roll_link: geometry collision mesh filename=package://legged_robot_mpc_controller/description/robots/g1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; visual mesh filename=package://legged_robot_mpc_controller/description/robots/g1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
- link left_wrist_yaw_link: geometry collision mesh filename=package://legged_robot_mpc_controller/description/robots/g1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; visual mesh filename=package://legged_robot_mpc_controller/description/robots/g1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
- link logo_link: geometry collision mesh filename=package://legged_robot_mpc_controller/description/robots/g1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; visual mesh filename=package://legged_robot_mpc_controller/description/robots/g1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
- link pelvis: geometry visual mesh filename=package://legged_robot_mpc_controller/description/robots/g1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
- link pelvis_contour_link: geometry collision mesh filename=package://legged_robot_mpc_controller/description/robots/g1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; visual mesh filename=package://legged_robot_mpc_controller/description/robots/g1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
- link right_ankle_pitch_link: geometry collision mesh filename=package://legged_robot_mpc_controller/description/robots/g1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; visual mesh filename=package://legged_robot_mpc_controller/description/robots/g1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
- link right_ankle_roll_link: geometry collision sphere radius=0.005; collision sphere radius=0.005
- link right_elbow_link: geometry collision mesh filename=package://legged_robot_mpc_controller/description/robots/g1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; visual mesh filename=package://legged_robot_mpc_controller/description/robots/g1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
- link right_hip_pitch_link: geometry collision mesh filename=package://legged_robot_mpc_controller/description/robots/g1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; visual mesh filename=package://legged_robot_mpc_controller/description/robots/g1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
- link right_hip_roll_link: geometry collision mesh filename=package://legged_robot_mpc_controller/description/robots/g1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; visual mesh filename=package://legged_robot_mpc_controller/description/robots/g1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
- link right_hip_yaw_link: geometry collision mesh filename=package://legged_robot_mpc_controller/description/robots/g1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; visual mesh filename=package://legged_robot_mpc_controller/description/robots/g1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
- link right_knee_link: geometry collision mesh filename=package://legged_robot_mpc_controller/description/robots/g1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; visual mesh filename=package://legged_robot_mpc_controller/description/robots/g1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
- link right_rubber_hand: geometry visual mesh filename=package://legged_robot_mpc_controller/description/robots/g1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
- link right_shoulder_pitch_link: geometry collision cylinder length=0.05 radius=0.03; visual mesh filename=package://legged_robot_mpc_controller/description/robots/g1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
- link right_shoulder_roll_link: geometry collision cylinder length=0.03 radius=0.03; visual mesh filename=package://legged_robot_mpc_controller/description/robots/g1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
- link right_shoulder_yaw_link: geometry collision mesh filename=package://legged_robot_mpc_controller/description/robots/g1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; visual mesh filename=package://legged_robot_mpc_controller/description/robots/g1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
- link right_wrist_pitch_link: geometry collision mesh filename=package://legged_robot_mpc_controller/description/robots/g1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; visual mesh filename=package://legged_robot_mpc_controller/description/robots/g1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
- link right_wrist_roll_link: geometry collision mesh filename=package://legged_robot_mpc_controller/description/robots/g1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; visual mesh filename=package://legged_robot_mpc_controller/description/robots/g1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
- link right_wrist_yaw_link: geometry collision mesh filename=package://legged_robot_mpc_controller/description/robots/g1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; visual mesh filename=package://legged_robot_mpc_controller/description/robots/g1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
- link torso_link: geometry collision mesh filename=package://legged_robot_mpc_controller/description/robots/g1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; visual mesh filename=package://legged_robot_mpc_controller/description/robots/g1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
- link waist_roll_link: geometry visual mesh filename=package://legged_robot_mpc_controller/description/robots/g1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
- link waist_yaw_link: geometry visual mesh filename=package://legged_robot_mpc_controller/description/robots/g1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
