Commit message: FEAT: unified RViz environment in env.urdf.xacro
env.urdf.xacro owns the world link and includes the terrain and object pieces,
commented or uncommented like the MuJoCo scene. Each piece attaches to world,
keeps its properties local and loads its own params by a relative path, so the
launch no longer needs environmentDescription or the params-file arguments and
always publishes env.urdf.xacro as /environment/robot_description.

Co-Authored-By: Claude Opus 5.5 <noreply@anthropic.com>

File: description/urdf/objects/boxes.urdf.xacro (robot description, xacro)
@@ -2,19 +2,14 @@
 <robot name="boxes" xmlns:xacro="http://www.ros.org/wiki/xacro">
   <!--
-    Environment description: the parametric boxes (same convention as
+    Environment piece: the parametric boxes (same convention as
     ../../mujoco/objects/boxes.xml.xacro, driven by the SAME params file). It is not
-    part of the robot. robot.launch.py runs it through xacro when selected with
-    environmentDescription and publishes it with its own robot_state_publisher in
-    the "environment" namespace.
+    part of the robot. Include it from ../env.urdf.xacro, which owns the "world" link.
     The boxes are free bodies in the simulator, so this shows their SPAWN pose:
-      <parent> -[fixed]-> <name of box 1> ... <name of box N>
+      world -[fixed]-> <name of box 1> ... <name of box N>
+    Everything sits inside a macro, so these properties stay local.
   -->
-  <xacro:arg name="boxes_params_file" default="../../../config/objects/boxes_params.yaml"/>
-  <xacro:arg name="parent" default="world"/>
-  <xacro:property name="boxes_params_file" value="$(arg boxes_params_file)"/>
-  <xacro:property name="parent_link"       value="$(arg parent)"/>
-  <xacro:property name="boxes" value="${xacro.load_yaml(boxes_params_file)['boxes']}"/>
+  <xacro:macro name="boxes_environment">
+  <xacro:property name="boxes" value="${xacro.load_yaml('../../../config/objects/boxes_params.yaml')['boxes']}"/>
   <xacro:property name="box_ids" value="${list(boxes.keys())}"/>
-  <link name="${parent_link}"/>
   <!--
     Recursively emit one link + fixed joint per box.
@@ -44,5 +39,5 @@
       </link>
       <joint name="${name}_joint" type="fixed">
-        <parent link="${parent_link}"/>
+        <parent link="world"/>
         <child link="${name}"/>
         <origin xyz="${p[0]} ${p[1]} ${p[2]}" rpy="0 0 ${box['yaw']}"/>
@@ -52,3 +47,5 @@
   </xacro:macro>
   <xacro:emit_box i="${0}"/>
+  </xacro:macro>
+  <xacro:boxes_environment/>
 </robot>

File: description/urdf/terrains/ramp.urdf.xacro (robot description, xacro)
@@ -2,21 +2,17 @@
 <robot name="ramp" xmlns:xacro="http://www.ros.org/wiki/xacro">
   <!--
-    Environment description: a parametric ramp (same geometry convention as
+    Environment piece: a parametric ramp (same geometry convention as
     ../../mujoco/terrains/ramp.xml.xacro, driven by the SAME params file). It is not
-    part of the robot. robot.launch.py runs it through xacro when selected with
-    environmentDescription and publishes it with its own robot_state_publisher in
-    the "environment" namespace, so rviz shows it next to the robot.
-    The result is a chain of fixed joints, rooted at <parent> (default "world"):
-      <parent> -[fixed]-> ramp_base -[fixed]-> ramp_wedge
+    part of the robot. Include it from ../env.urdf.xacro, which owns the "world" link.
+    The result is a chain of fixed joints, rooted at "world":
+      world -[fixed]-> ramp_base -[fixed]-> ramp_wedge
     The "ramp_base" link is the entry-edge reference frame (world pos + yaw).
     URDF has no wedge primitive, so the wedge is the unit mesh
     description/meshes/terrains/unit_wedge.stl (x in [0, 1], y in [-0.5, 0.5],
     top rising from z = 0 to z = 1) scaled by (length, width, rise).
+    Everything sits inside a macro, so these properties stay local.
   -->
-  <xacro:arg name="ramp_params_file" default="../../../config/terrains/ramp_params.yaml"/>
-  <xacro:arg name="parent" default="world"/>
-  <xacro:property name="ramp_params_file" value="$(arg ramp_params_file)"/>
-  <xacro:property name="parent_link"      value="$(arg parent)"/>
-  <xacro:property name="ramp" value="${xacro.load_yaml(ramp_params_file)['ramp']}"/>
+  <xacro:macro name="ramp_environment">
+  <xacro:property name="ramp" value="${xacro.load_yaml('../../../config/terrains/ramp_params.yaml')['ramp']}"/>
   <xacro:property name="base"    value="${ramp['base']}"/>
   <xacro:property name="L"       value="${ramp['length']}"/>
@@ -25,9 +21,8 @@
   <xacro:property name="gray"    value="${ramp['color_gray']}"/>
   <xacro:property name="mesh"    value="package://legged_robot_mpc_controller/description/meshes/terrains/unit_wedge.stl"/>
-  <link name="${parent_link}"/>
   <!-- Entry-edge reference frame: world position + yaw. -->
   <link name="ramp_base"/>
   <joint name="ramp_base_joint" type="fixed">
-    <parent link="${parent_link}"/>
+    <parent link="world"/>
     <child link="ramp_base"/>
     <origin xyz="${base['pos'][0]} ${base['pos'][1]} ${base['pos'][2]}"
@@ -55,3 +50,5 @@
     <child link="ramp_wedge"/>
   </joint>
+  </xacro:macro>
+  <xacro:ramp_environment/>
 </robot>

File: description/urdf/terrains/stairs.urdf.xacro (robot description, xacro)
@@ -2,20 +2,17 @@
 <robot name="stairs" xmlns:xacro="http://www.ros.org/wiki/xacro">
   <!--
-    Environment description: a parametric staircase (same geometry convention
-    as ../../mujoco/terrains/stairs.xml.xacro, driven by the SAME params file). It is not
-    part of the robot. robot.launch.py runs it through xacro and publishes it with
-    its own robot_state_publisher in the "environment" namespace, so rviz shows
-    it next to the robot.
-    The result is a chain of fixed joints, rooted at <parent> (default "world"):
-      <parent> -[fixed]-> stairs_base -[fixed]-> stairs_step_1 ... stairs_step_N
+    Environment piece: a parametric staircase (same geometry convention as
+    ../../mujoco/terrains/stairs.xml.xacro, driven by the SAME params file). It is not
+    part of the robot. Include it from ../env.urdf.xacro, which owns the "world" link;
+    robot.launch.py publishes that file as /environment/robot_description for rviz.
+    The result is a chain of fixed joints, rooted at "world":
+      world -[fixed]-> stairs_base -[fixed]-> stairs_step_1 ... stairs_step_N
     The "stairs_base" link is the 0th step reference frame (world pos + yaw).
     Each step is a SOLID box from the ground up to its tread height; the box
-    origin sits at half that height.
+    origin sits at half that height. Everything sits inside a macro, so these
+    properties stay local and do not collide with other included pieces.
   -->
-  <xacro:arg name="stairs_params_file" default="../../../config/terrains/stairs_params.yaml"/>
-  <xacro:arg name="parent" default="world"/>
-  <xacro:property name="stairs_params_file" value="$(arg stairs_params_file)"/>
-  <xacro:property name="parent_link"        value="$(arg parent)"/>
-  <xacro:property name="stairs" value="${xacro.load_yaml(stairs_params_file)['stairs']}"/>
+  <xacro:macro name="stairs_environment">
+  <xacro:property name="stairs" value="${xacro.load_yaml('../../../config/terrains/stairs_params.yaml')['stairs']}"/>
   <xacro:property name="base"      value="${stairs['base']}"/>
   <xacro:property name="num_steps" value="${stairs['num_steps']}"/>
@@ -26,9 +23,8 @@
   <xacro:property name="gray_step" value="${stairs['color_gray_step']}"/>
   <xacro:property name="gray_max"  value="${stairs['color_gray_max']}"/>
-  <link name="${parent_link}"/>
   <!-- 0th step reference frame: world center position + yaw. -->
   <link name="stairs_base"/>
   <joint name="stairs_base_joint" type="fixed">
-    <parent link="${parent_link}"/>
+    <parent link="world"/>
     <child link="stairs_base"/>
     <origin xyz="${base['pos'][0]} ${base['pos'][1]} ${base['pos'][2]}"
@@ -74,3 +70,5 @@
   </xacro:macro>
   <xacro:emit_step i="${1}" x0="${base['start_offset']}" z0="${0}"/>
+  </xacro:macro>
+  <xacro:stairs_environment/>
 </robot>

File: description/urdf/terrains/uneven_terrain.urdf.xacro (robot description, xacro)
@@ -1,5 +1,4 @@
 <robot name="uneven_terrain">
-  <!-- Generated by generate_uneven_terrain.py from shared YAML; xacro-compatible URDF. -->
-  <link name="world" />
+  <!-- Generated by generate_uneven_terrain.py from shared YAML. Include it from ../env.urdf.xacro, which owns the world link. -->
   <link name="uneven_terrain">
     <visual name="terrain_000_000_0">
